Commit message: updated monkey_complete.urdf

File: monkey_complete/urdf/monkey_complete.urdf (robot description, URDF)
Before this commit: robot monkey_co mplete, 15 links, 14 joints
Links:
- added link world
Joints:
- added joint world_to_base_link=: type fixed, parent world, child base_link
- joint L_Ellbow_Joint: limit lower=-1.507 upper=1.507 effort=1 velocity=1 -> lower=-1.4 upper=0 effort=1 velocity=1
- joint L_Shoulder_Fro_Joint: axis -1 0 0 -> 1 0 0; limit lower=-1.507 upper=1.507 effort=1 velocity=1 -> lower=-2.186 upper=0.615 effort=1 velocity=1
- joint L_Shoulder_Hor_Joint: limit lower=-1.507 upper=1.507 effort=1 velocity=1 -> lower=-1.2 upper=1.6 effort=1 velocity=1
- joint L_Shoulder_Lat_Joint: limit lower=-1.507 upper=1.507 effort=1 velocity=1 -> lower=-1.4 upper=1.4 effort=1 velocity=1
- joint L_Wrist_Joint: limit lower=-1.507 upper=1.507 effort=1 velocity=1 -> lower=-1.4 upper=1.4 effort=1 velocity=1
- joint Neck_Fro_Rot_Joint: limit lower=-1.507 upper=1.507 effort=1 velocity=1 -> lower=-1.4 upper=1.4 effort=1 velocity=1
- joint Neck_Hor_Rot_Joint: axis 0 0 -1 -> 0 0 1; limit lower=-1.507 upper=1.507 effort=1 velocity=1 -> lower=-1.4 upper=1.4 effort=1 velocity=1
- joint R_Ellbow_Joint: limit lower=-1.507 upper=1.507 effort=1 velocity=1 -> lower=0 upper=1.4 effort=1 velocity=1
- joint R_Shoulder_Fro_Rot_Joint: limit lower=-1.507 upper=1.507 effort=1 velocity=1 -> lower=-2.186 upper=0.615 effort=1 velocity=1
- joint R_Shoulder_Hor_Joint: limit lower=-1.507 upper=1.507 effort=1 velocity=1 -> lower=-1.6 upper=1.2 effort=1 velocity=1
- joint R_Shoulder_Lat_Joint: limit lower=-1.507 upper=1.507 effort=1 velocity=1 -> lower=-1.4 upper=1.4 effort=1 velocity=1
- joint R_Wrist_Joint: limit lower=-1.507 upper=1.507 effort=1 velocity=1 -> lower=-1.4 upper=1.4 effort=1 velocity=1

Commit message: faster

File: monkey_complete/urdf/monkey_complete.urdf (robot description, URDF)
Before this commit: robot monkey_robot, 16 links, 15 joints
Joints:
- joint L_Ellbow_Joint: limit lower=-1.4 upper=0 effort=1 velocity=1 -> lower=-1.4 upper=0 effort=1 velocity=5
- joint L_Shoulder_Fro_Joint: limit lower=-2.186 upper=0.615 effort=1 velocity=1 -> lower=-2.186 upper=0.615 effort=1 velocity=5
- joint L_Shoulder_Hor_Joint: limit lower=-1.2 upper=1.6 effort=1 velocity=1 -> lower=-1.2 upper=1.6 effort=1 velocity=5
- joint L_Shoulder_Lat_Joint: limit lower=-1.4 upper=1.4 effort=1 velocity=1 -> lower=-1.4 upper=1.4 effort=1 velocity=5
- joint L_Wrist_Joint: limit lower=-1.4 upper=1.4 effort=1 velocity=1 -> lower=-1.4 upper=1.4 effort=1 velocity=5
- joint Neck_Fro_Rot_Joint: limit lower=-1.4 upper=1.4 effort=1 velocity=1 -> lower=-1.4 upper=1.4 effort=1 velocity=5
- joint Neck_Hor_Rot_Joint: limit lower=-1.4 upper=1.4 effort=1 velocity=1 -> lower=-1.4 upper=1.4 effort=1 velocity=5
- joint R_Ellbow_Joint: limit lower=0 upper=1.4 effort=1 velocity=1 -> lower=0 upper=1.4 effort=1 velocity=5
- joint R_Shoulder_Fro_Rot_Joint: limit lower=-2.186 upper=0.615 effort=1 velocity=1 -> lower=-2.186 upper=0.615 effort=1 velocity=5
- joint R_Shoulder_Hor_Joint: limit lower=-1.6 upper=1.2 effort=1 velocity=1 -> lower=-1.6 upper=1.2 effort=1 velocity=5
- joint R_Shoulder_Lat_Joint: limit lower=-1.4 upper=1.4 effort=1 velocity=1 -> lower=-1.4 upper=1.4 effort=1 velocity=5
- joint R_Wrist_Joint: limit lower=-1.4 upper=1.4 effort=1 velocity=1 -> lower=-1.4 upper=1.4 effort=1 velocity=5

Commit message: faster

File: monkey_complete/urdf/monkey_complete.urdf (robot description, URDF)
Before this commit: robot monkey_robot, 16 links, 15 joints
Joints:
- joint L_Ellbow_Joint: limit lower=-1.4 upper=0 effort=1 velocity=5 -> lower=-1.4 upper=0 effort=1 velocity=20
- joint L_Shoulder_Fro_Joint: limit lower=-2.186 upper=0.615 effort=1 velocity=5 -> lower=-2.186 upper=0.615 effort=1 velocity=20
- joint L_Shoulder_Hor_Joint: limit lower=-1.2 upper=1.6 effort=1 velocity=5 -> lower=-1.2 upper=1.6 effort=1 velocity=20
- joint L_Shoulder_Lat_Joint: limit lower=-1.4 upper=1.4 effort=1 velocity=5 -> lower=-1.4 upper=1.4 effort=1 velocity=20
- joint L_Wrist_Joint: limit lower=-1.4 upper=1.4 effort=1 velocity=5 -> lower=-1.4 upper=1.4 effort=1 velocity=20
- joint Neck_Fro_Rot_Joint: limit lower=-1.4 upper=1.4 effort=1 velocity=5 -> lower=-1.4 upper=1.4 effort=1 velocity=20
- joint Neck_Hor_Rot_Joint: limit lower=-1.4 upper=1.4 effort=1 velocity=5 -> lower=-1.4 upper=1.4 effort=1 velocity=20
- joint R_Ellbow_Joint: limit lower=0 upper=1.4 effort=1 velocity=5 -> lower=0 upper=1.4 effort=1 velocity=20
- joint R_Shoulder_Fro_Rot_Joint: limit lower=-2.186 upper=0.615 effort=1 velocity=5 -> lower=-2.186 upper=0.615 effort=1 velocity=20
- joint R_Shoulder_Hor_Joint: limit lower=-1.6 upper=1.2 effort=1 velocity=5 -> lower=-1.6 upper=1.2 effort=1 velocity=20
- joint R_Shoulder_Lat_Joint: limit lower=-1.4 upper=1.4 effort=1 velocity=5 -> lower=-1.4 upper=1.4 effort=1 velocity=20
- joint R_Wrist_Joint: limit lower=-1.4 upper=1.4 effort=1 velocity=5 -> lower=-1.4 upper=1.4 effort=1 velocity=20
